Commit message: Fix right wheel direction in diff_drive_example
Invert the right wheel joint axis to account for opposite mounting
direction. This ensures both wheels spin in the correct direction
for forward motion.

Co-Authored-By: Claude Opus 4.5 <noreply@anthropic.com>

File: src/diff_drive_example/urdf/diff_drive.urdf.xacro (robot description, xacro)
@@ -99,5 +99,5 @@
     <child link="right_wheel_link"/>
     <origin xyz="0 ${-wheel_separation/2} ${wheel_radius}" rpy="${-pi/2} 0 0"/>
-    <axis xyz="0 0 1"/>
+    <axis xyz="0 0 -1"/>
   </joint>
   <!-- Front caster wheel (for stability) -->
